File: CircularControllerLEDs/CircularControllerLEDs.brd (EAGLE design)
At the start: 88.6 x 95 mm, 21 parts

Commit message: Updated PCBs
Parts:
- R6, R8: device SparkFun-Resistors:0603-RES@1 -> SparkFun-Resistors:1206
- moved R6 1.52 mm to (75.2, 42.4)
- moved R8 1.52 mm to (75.2, 45.0)
- moved C3 1.05 mm to (9.40, 56.9)
- moved C2 0.25 mm to (73.3, 51.5)
Routing:
- net GND: track 0.00 -> 439.1 mm
- net 5V: track 83.1 -> 55.7 mm
- net VCC: track 283.4 -> 299.3 mm
- net N$3: track 13.3 -> 11.2 mm
- net N$1: track 9.10 -> 7.02 mm
- net LEDS_DI: track 3.21 -> 4.19 mm
- net LEDS_CI: track 3.21 -> 4.19 mm
- removed copper zone on layer 1, net GND
