File: CircularControllerLEDs/CircularControllerLEDs.sch (EAGLE design)
At the start: 21 parts

Commit message: Updated PCBs
Parts:
- R6, R8: device SparkFun-Resistors:220OHM-1/10W-1%(0603) -> SparkFun-Resistors:RESISTOR1206
Changed lines of the file:
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@@
 <part name="SUPPLY3" library="SparkFun-Aesthetics" deviceset="VCC" device=""/>
 <part name="GND5" library="SparkFun-Aesthetics" deviceset="GND" device=""/>
-<part name="R8" library="SparkFun-Resistors" deviceset="220OHM-1/10W-1%(0603)" device="" value="220"/>
+<part name="R8" library="SparkFun-Resistors" deviceset="RESISTOR" device="1206" value="220"/>
 <part name="GND3" library="SparkFun-Aesthetics" deviceset="GND" device=""/>
-<part name="R6" library="SparkFun-Resistors" deviceset="220OHM-1/10W-1%(0603)" device="" value="220"/>
+<part name="R6" library="SparkFun-Resistors" deviceset="RESISTOR" device="1206" value="220"/>
 <part name="SUPPLY4" library="SparkFun-Aesthetics" deviceset="VCC" device=""/>
 <part name="GND1" library="SparkFun-Aesthetics" deviceset="GND" device=""/>
